Commit message: Made changes to the URDF file which means that the robot is able to move now albeit erratically.

File: src/ford_bot/description/robot_core.xacro (robot description, xacro)
@@ -2,18 +2,46 @@
 <robot xmlns:xacro="http://www.ros.org/wiki/xacro" name="ford_robot">
     <xacro:include filename="inertial_macros.xacro"/>
-    <link name="world"/>
+    <material name="white">
+        <color rgba="1 1 1 1" />
+    </material>
+    <material name="orange">
+        <color rgba="1 0.3 0.1 1"/>
+    </material>
+    <material name="blue">
+        <color rgba="0.2 0.2 1 1"/>
+    </material>
+    <material name="black">
+        <color rgba="0 0 0 1"/>
+    </material>
+    <material name="red">
+        <color rgba="1 0 0 1"/>
+    </material>
+    <!-- BASE LINK -->
     <link name="base_link">
-        <visual name="">
-            <origin xyz="0.0 0.0 0.0" rpy="0.0 0.0 0.0"/>
+    </link>
+    <!-- BASE_FOOTPRINT LINK -->
+    <joint name="base_footprint_joint" type="fixed">
+        <parent link="base_link"/>
+        <child link="base_footprint"/>
+        <origin xyz="0 0 0" rpy="0 0 0"/>
+    </joint>
+    <link name="base_footprint">
+    </link>
+    <!-- CHASSIS LINK -->
+    <joint name="chassis_joint" type="fixed">
+        <parent link="base_link"/>
+        <child link="chassis"/>
+        <origin xyz="0.0 0.0 0.15"/>
+    </joint>
+    <link name="chassis">
+        <visual>
+            <origin xyz="0.0 0.0 0.0"/>
             <geometry>
                 <box size="0.7 0.6 0.1"/>
             </geometry>
-            <material name="">
-                <color rgba="1.0 0.0 0.0 1.0"/>
-                <texture filename=""/>
-            </material>
+            <material name="orange"/>
         </visual>
         <collision>
-            <origin xyz="0.0 0.0 0.0" rpy="0.0 0.0 0.0"/>
+            <origin xyz="0.0 0.0 0.0"/>
             <geometry>
                 <box size="0.7 0.6 0.1"/>
@@ -24,17 +52,10 @@
         </xacro:inertial_box>
     </link>
-    <gazebo reference="base_link"> <!-- reference to a existing "link" -->
-        <material>Gazebo/Red</material>
-        <selfCollide>True</selfCollide>
+    <gazebo reference="chassis">
+        <material>Gazebo/Orange</material>
     </gazebo>
-    <joint name="base_joint" type="fixed">
-        <origin xyz="0.0 0.0 0.135" rpy="0.0 0.0 0.0"/>
-        <parent link="world"/>
-        <child link="base_link"/>
-        <axis xyz="0.0 0.0 0.0"/>
-    </joint>
-    <!-- All Wheel links and joints -->
+       <!-- All Wheel links and joints -->
     <xacro:macro name="wheel" params="name x y z">
-        <link name="${name}_wheel_link">
+        <link name="${name}_wheel">
             <visual name="">
                 <origin xyz="0.0 0.0 0.0" rpy="1.57 0.0 0.0"/>
@@ -56,41 +77,29 @@
             </xacro:inertial_cylinder>
         </link>
-        <!-- <gazebo reference="${name}_wheel_link">
-            <material>Gazebo/Yellow</material>
-        </gazebo> -->
         <joint name="${name}_wheel_joint" type="continuous">
             <origin xyz="${x} ${y} ${z}" rpy="0 0.0 0.0"/>
-            <parent link="base_link"/>
-            <child link="${name}_wheel_link"/>
-            <limit effort="100" lower="-3.14" upper="3.14" velocity="1.0"/>
+            <parent link="chassis"/>
+            <child link="${name}_wheel"/>
+            <limit effort="1000.0" velocity="1.0"/>
             <axis xyz=".0 1.0 0.0"/>
         </joint>
-        <!-- This block provides the simulator (Gazebo) with information on a few additional
-        physical properties. See http://gazebosim.org/tutorials/?tut=ros_urdf for more-->
-        <gazebo reference="${name}_wheel_link">
-            <mu1 value="200.0"/>
-            <mu2 value="100.0"/>
-            <kp value="10000000.0" />
-            <kd value="1.0" />
-            <material>Gazebo/Grey</material>
-        </gazebo>
-    <!-- This block connects the wheel joint to an actuator (motor), which informs both
+            <!-- This block connects the wheel joint to an actuator (motor), which informs both
     simulation and visualization of the robot -->
-    <transmission name="${name}_wheel_trans">
-      <type>transmission_interface/SimpleTransmission</type>
-      <actuator name="${name}_wheel_motor">
-        <hardwareInterface>hardware_interface/VelocityJointInterface</hardwareInterface>
-        <mechanicalReduction>1</mechanicalReduction>
-      </actuator>
-      <joint name="${name}_wheel_joint">
-        <hardwareInterface>hardware_interface/VelocityJointInterface</hardwareInterface>
-      </joint>
-    </transmission>
+        <transmission name="${name}_wheel_transmission">
+        <type>transmission_interface/SimpleTransmission</type>
+        <actuator name="${name}_wheel_actuator">
+            <hardwareInterface>hardware_interface/EffortJointInterface</hardwareInterface>
+            <mechanicalReduction>1</mechanicalReduction>
+        </actuator>
+        <joint name="${name}_wheel_joint">
+            <hardwareInterface>hardware_interface/EffortJointInterface</hardwareInterface>
+        </joint>
+        </transmission>
     </xacro:macro>
     <!-- Wheel Creating using macros -->
-    <xacro:wheel name="front_left"  x="0.250" y ="0.325" z="-0.035"/>
-    <xacro:wheel name="rear_left" x="-0.250" y ="0.325" z="-0.035"/>
-    <xacro:wheel name="front_right"  x="0.250" y ="-0.325" z="-0.035"/>
-    <xacro:wheel name="rear_right"   x="-0.250" y =" -0.325" z="-0.035"/>
+    <xacro:wheel name="front_left"  x="0.250" y ="0.325" z="-0.055"/>
+    <xacro:wheel name="rear_left" x="-0.250" y ="0.325" z="-0.055"/>
+    <xacro:wheel name="front_right"  x="0.250" y ="-0.325" z="-0.055"/>
+    <xacro:wheel name="rear_right"   x="-0.250" y ="-0.325" z="-0.055"/>
     <gazebo>
         <plugin name="gazebo_ros_control" filename="libgazebo_ros_control.so">
@@ -99,42 +108,3 @@
         </plugin>
     </gazebo>
-    <!-- <transmission name="${prefix}_${suffix}_wheel_trans">
-      <type>transmission_interface/SimpleTransmission</type>
-      <actuator name="${prefix}_${suffix}_wheel_motor">
-        <mechanicalReduction>1</mechanicalReduction>
-      </actuator>
-      <joint name="${prefix}_${suffix}_wheel_joint">
-        <hardwareInterface>VelocityJointInterface</hardwareInterface>
-      </joint>
-    </transmission>
-    <transmission name="tran2">
-        <type>transmission_interface/SimpleTransmission</type>
-        <joint name="front_right_wheel_joint">
-            <hardwareInterface>hardware_interface/EffortJointInterface</hardwareInterface>
-        </joint>
-        <actuator name="motor2">
-            <hardwareInterface>hardware_interface/EffortJointInterface</hardwareInterface>
-            <mechanicalReduction>1</mechanicalReduction>
-        </actuator>
-    </transmission>
-    <transmission name="tran3">
-        <type>transmission_interface/SimpleTransmission</type>
-        <joint name="rear_left_wheel_joint">
-            <hardwareInterface>hardware_interface/EffortJointInterface</hardwareInterface>
-        </joint>
-        <actuator name="motor3">
-            <hardwareInterface>hardware_interface/EffortJointInterface</hardwareInterface>
-            <mechanicalReduction>1</mechanicalReduction>
-        </actuator>
-    </transmission>
-    <transmission name="tran4">
-        <type>transmission_interface/SimpleTransmission</type>
-        <joint name="front_left_wheel_joint">
-            <hardwareInterface>hardware_interface/EffortJointInterface</hardwareInterface>
-        </joint>
-        <actuator name="motor4">
-            <hardwareInterface>hardware_interface/EffortJointInterface</hardwareInterface>
-            <mechanicalReduction>1</mechanicalReduction>
-        </actuator>
-    </transmission> -->
 </robot>

Commit message: The robot is now stable after making changes to the PID controller in the movement.yaml file. Combined the launch file for the robot and the controllers into one so it all starts together now.

File: src/ford_bot/description/robot_core.xacro (robot description, xacro)
@@ -18,9 +18,9 @@
     </material>
     <!-- BASE LINK -->
-    <link name="base_link">
+    <link name="base">
     </link>
     <!-- BASE_FOOTPRINT LINK -->
     <joint name="base_footprint_joint" type="fixed">
-        <parent link="base_link"/>
+        <parent link="base"/>
         <child link="base_footprint"/>
         <origin xyz="0 0 0" rpy="0 0 0"/>
@@ -30,5 +30,5 @@
     <!-- CHASSIS LINK -->
     <joint name="chassis_joint" type="fixed">
-        <parent link="base_link"/>
+        <parent link="base_footprint"/>
         <child link="chassis"/>
         <origin xyz="0.0 0.0 0.15"/>
@@ -40,5 +40,5 @@
                 <box size="0.7 0.6 0.1"/>
             </geometry>
-            <material name="orange"/>
+            <material name="red"/>
         </visual>
         <collision>
@@ -53,5 +53,5 @@
     </link>
     <gazebo reference="chassis">
-        <material>Gazebo/Orange</material>
+        <material>Gazebo/Red</material>
     </gazebo>
        <!-- All Wheel links and joints -->
@@ -63,5 +63,5 @@
                     <cylinder radius="0.1" length="0.05"/>
                 </geometry>
-                <material name="black">
+                <material name="white">
                     <color rgba="1.0 1.0 0.0 1.0"/>
                 </material>
@@ -77,9 +77,12 @@
             </xacro:inertial_cylinder>
         </link>
+        <gazebo reference="${name}_wheel">
+            <material>Gazebo/White</material>
+        </gazebo>
         <joint name="${name}_wheel_joint" type="continuous">
             <origin xyz="${x} ${y} ${z}" rpy="0 0.0 0.0"/>
             <parent link="chassis"/>
             <child link="${name}_wheel"/>
-            <limit effort="1000.0" velocity="1.0"/>
+            <limit effort="1000.0" velocity="5.0"/>
             <axis xyz=".0 1.0 0.0"/>
         </joint>

Commit message: made changes to the robot urdf file to include a skid steer drive plugin which now enables the use to move and control the robot using the keyboard by simply running the teleop_twist node and python script.

File: src/ford_bot/description/robot_core.xacro (robot description, xacro)
@@ -2,4 +2,5 @@
 <robot xmlns:xacro="http://www.ros.org/wiki/xacro" name="ford_robot">
     <xacro:include filename="inertial_macros.xacro"/>
+    <xacro:include filename="gazebo_params.xacro"/>
     <material name="white">
         <color rgba="1 1 1 1" />
@@ -52,7 +53,13 @@
         </xacro:inertial_box>
     </link>
+<!--
     <gazebo reference="chassis">
+        <mu1>0.2</mu1>
+        <mu2>0.2</mu2>
         <material>Gazebo/Red</material>
-    </gazebo>
+    </gazebo> -->
+    <!-- <gazebo reference="chassis">
+        <material>Gazebo/Red</material>
+    </gazebo> -->
        <!-- All Wheel links and joints -->
     <xacro:macro name="wheel" params="name x y z">
@@ -77,7 +84,12 @@
             </xacro:inertial_cylinder>
         </link>
-        <gazebo reference="${name}_wheel">
+        <!-- <gazebo reference="${name}_wheel">
+            <mu1>0.2</mu1>
+            <mu2>0.2</mu2>
+            <material>Gazebo/Yellow</material>
+        </gazebo> -->
+        <!-- <gazebo reference="${name}_wheel">
             <material>Gazebo/White</material>
-        </gazebo>
+        </gazebo> -->
         <joint name="${name}_wheel_joint" type="continuous">
             <origin xyz="${x} ${y} ${z}" rpy="0 0.0 0.0"/>
@@ -89,5 +101,5 @@
             <!-- This block connects the wheel joint to an actuator (motor), which informs both
     simulation and visualization of the robot -->
-        <transmission name="${name}_wheel_transmission">
+        <!-- <transmission name="${name}_wheel_transmission">
         <type>transmission_interface/SimpleTransmission</type>
         <actuator name="${name}_wheel_actuator">
@@ -98,5 +110,5 @@
             <hardwareInterface>hardware_interface/EffortJointInterface</hardwareInterface>
         </joint>
-        </transmission>
+        </transmission> -->
     </xacro:macro>
     <!-- Wheel Creating using macros -->
@@ -105,9 +117,10 @@
     <xacro:wheel name="front_right"  x="0.250" y ="-0.325" z="-0.055"/>
     <xacro:wheel name="rear_right"   x="-0.250" y ="-0.325" z="-0.055"/>
-    <gazebo>
+    <!-- <gazebo>
         <plugin name="gazebo_ros_control" filename="libgazebo_ros_control.so">
             <robotNamespace>/ford_robot</robotNamespace>
             <robotSimType>gazebo_ros_control/DefaultRobotHWSim</robotSimType>
+            <commandTopic>cmd_vel</commandTopic>
         </plugin>
-    </gazebo>
+    </gazebo> -->
 </robot>
