Commit message: Added a lidar to the robot.

File: src/ford_bot/description/ford_robot.urdf.xacro (robot description, xacro)
@@ -2,3 +2,4 @@
 <robot xmlns:xacro="http://www.ros.org/wiki/xacro" name="ford_robot">
     <xacro:include filename="$(find ford_bot)/description/robot_core.xacro"/>
+    <xacro:include filename="$(find ford_bot)/description/lidar.xacro"/>
 </robot>

File: src/ford_bot/description/gazebo_params.xacro (robot description, xacro)
@@ -4,25 +4,25 @@
 <mu1>0.2</mu1>
 <mu2>0.2</mu2>
-<material>Gazebo/Red</material>
+<material>Gazebo/Green</material>
 </gazebo>
 <gazebo reference="front_right_wheel">
 <mu1>0.2</mu1>
 <mu2>0.2</mu2>
-<material>Gazebo/Yellow</material>
+<material>Gazebo/White</material>
 </gazebo>
 <gazebo reference="front_left_wheel">
 <mu1>0.2</mu1>
 <mu2>0.2</mu2>
-<material>Gazebo/Yellow</material>
+<material>Gazebo/White</material>
 </gazebo>
 <gazebo reference="rear_right_wheel">
 <mu1>0.2</mu1>
 <mu2>0.2</mu2>
-<material>Gazebo/Yellow</material>
+<material>Gazebo/White</material>
 </gazebo>
 <gazebo reference="rear_left_wheel">
 <mu1>0.2</mu1>
 <mu2>0.2</mu2>
-<material>Gazebo/Yellow</material>
+<material>Gazebo/White</material>
 </gazebo>
 <!-- Controller for the 4-wheeled robot -->
@@ -46,5 +46,5 @@
         <odometryTopic>odom</odometryTopic>
         <odometryFrame>odom</odometryFrame>
-        <robotBaseFrame>base</robotBaseFrame>
+        <robotBaseFrame>base_footprint</robotBaseFrame>
         <publishWheelTF>true</publishWheelTF>
         <publishOdom>true</publishOdom>

File: src/ford_bot/description/robot_core.xacro (robot description, xacro)
@@ -53,13 +53,4 @@
         </xacro:inertial_box>
     </link>
-<!--
-    <gazebo reference="chassis">
-        <mu1>0.2</mu1>
-        <mu2>0.2</mu2>
-        <material>Gazebo/Red</material>
-    </gazebo> -->
-    <!-- <gazebo reference="chassis">
-        <material>Gazebo/Red</material>
-    </gazebo> -->
        <!-- All Wheel links and joints -->
     <xacro:macro name="wheel" params="name x y z">
@@ -84,12 +75,4 @@
             </xacro:inertial_cylinder>
         </link>
-        <!-- <gazebo reference="${name}_wheel">
-            <mu1>0.2</mu1>
-            <mu2>0.2</mu2>
-            <material>Gazebo/Yellow</material>
-        </gazebo> -->
-        <!-- <gazebo reference="${name}_wheel">
-            <material>Gazebo/White</material>
-        </gazebo> -->
         <joint name="${name}_wheel_joint" type="continuous">
             <origin xyz="${x} ${y} ${z}" rpy="0 0.0 0.0"/>
@@ -99,16 +82,4 @@
             <axis xyz=".0 1.0 0.0"/>
         </joint>
-            <!-- This block connects the wheel joint to an actuator (motor), which informs both
-    simulation and visualization of the robot -->
-        <!-- <transmission name="${name}_wheel_transmission">
-        <type>transmission_interface/SimpleTransmission</type>
-        <actuator name="${name}_wheel_actuator">
-            <hardwareInterface>hardware_interface/EffortJointInterface</hardwareInterface>
-            <mechanicalReduction>1</mechanicalReduction>
-        </actuator>
-        <joint name="${name}_wheel_joint">
-            <hardwareInterface>hardware_interface/EffortJointInterface</hardwareInterface>
-        </joint>
-        </transmission> -->
     </xacro:macro>
     <!-- Wheel Creating using macros -->
@@ -117,10 +88,3 @@
     <xacro:wheel name="front_right"  x="0.250" y ="-0.325" z="-0.055"/>
     <xacro:wheel name="rear_right"   x="-0.250" y ="-0.325" z="-0.055"/>
-    <!-- <gazebo>
-        <plugin name="gazebo_ros_control" filename="libgazebo_ros_control.so">
-            <robotNamespace>/ford_robot</robotNamespace>
-            <robotSimType>gazebo_ros_control/DefaultRobotHWSim</robotSimType>
-            <commandTopic>cmd_vel</commandTopic>
-        </plugin>
-    </gazebo> -->
 </robot>

Commit message: Added a new implementation of the lidar gazebo parameters and now it shows the laserScan messages in RViz. However the robot won't move in RViz but it does operate as expected in Gazebo.

File: src/ford_bot/description/ford_robot.urdf.xacro (robot description, xacro)
@@ -2,4 +2,5 @@
 <robot xmlns:xacro="http://www.ros.org/wiki/xacro" name="ford_robot">
     <xacro:include filename="$(find ford_bot)/description/robot_core.xacro"/>
+    <!-- <xacro:include filename="$(find ford_bot)/description/test_robot.xacro"/> -->
     <xacro:include filename="$(find ford_bot)/description/lidar.xacro"/>
 </robot>

File: src/ford_bot/description/gazebo_params.xacro (robot description, xacro)
@@ -1,57 +1,57 @@
 <?xml version="1.0"?>
 <robot xmlns:xacro="http://www.ros.org/wiki/xacro">
-<gazebo reference="chassis">
-<mu1>0.2</mu1>
-<mu2>0.2</mu2>
-<material>Gazebo/Green</material>
-</gazebo>
-<gazebo reference="front_right_wheel">
-<mu1>0.2</mu1>
-<mu2>0.2</mu2>
-<material>Gazebo/White</material>
-</gazebo>
-<gazebo reference="front_left_wheel">
-<mu1>0.2</mu1>
-<mu2>0.2</mu2>
-<material>Gazebo/White</material>
-</gazebo>
-<gazebo reference="rear_right_wheel">
-<mu1>0.2</mu1>
-<mu2>0.2</mu2>
-<material>Gazebo/White</material>
-</gazebo>
-<gazebo reference="rear_left_wheel">
-<mu1>0.2</mu1>
-<mu2>0.2</mu2>
-<material>Gazebo/White</material>
-</gazebo>
+    <gazebo reference="chassis">
+        <mu1>0.2</mu1>
+        <mu2>0.2</mu2>
+        <material>Gazebo/Green</material>
+    </gazebo>
+    <gazebo reference="front_right_wheel">
+        <mu1>0.2</mu1>
+        <mu2>0.2</mu2>
+        <material>Gazebo/White</material>
+    </gazebo>
+    <gazebo reference="front_left_wheel">
+        <mu1>0.2</mu1>
+        <mu2>0.2</mu2>
+        <material>Gazebo/White</material>
+    </gazebo>
+    <gazebo reference="rear_right_wheel">
+        <mu1>0.2</mu1>
+        <mu2>0.2</mu2>
+        <material>Gazebo/White</material>
+    </gazebo>
+    <gazebo reference="rear_left_wheel">
+        <mu1>0.2</mu1>
+        <mu2>0.2</mu2>
+        <material>Gazebo/White</material>
+    </gazebo>
 <!-- Controller for the 4-wheeled robot -->
-<gazebo>
-    <plugin name="skid_steer_drive_controller" filename="libgazebo_ros_skid_steer_drive.so">
-        <!-- Control update rate in Hz -->
-        <updateRate>100.0</updateRate>
-        <!-- Leave empty otherwise there will be problems with sending control commands -->
-        <robotNamespace> </robotNamespace>
-        <!-- Robot kinematics -->
-        <leftFrontJoint>front_left_wheel_joint</leftFrontJoint>
-        <rightFrontJoint>front_right_wheel_joint</rightFrontJoint>
-        <leftRearJoint>rear_left_wheel_joint</leftRearJoint>
-        <rightRearJoint>rear_right_wheel_joint</rightRearJoint>
-        <wheelSeparation>0.65</wheelSeparation>
-        <wheelDiameter>0.2</wheelDiameter>
-        <!-- Maximum torque which the wheels can produce, in Nm, defaults to 5 Nm -->
-        <torque>1000</torque>
-        <!-- Topic to reveive -->
-        <commandTopic>cmd_vel</commandTopic>
-        <odometryTopic>odom</odometryTopic>
-        <odometryFrame>odom</odometryFrame>
-        <robotBaseFrame>base_footprint</robotBaseFrame>
-        <publishWheelTF>true</publishWheelTF>
-        <publishOdom>true</publishOdom>
-        <publishJointState>true</publishJointState>
-        <covariance_x>0.0001</covariance_x>
-        <covariance_y>0.0001</covariance_y>
-        <covariance_yaw>0.01</covariance_yaw>
-    </plugin>
-</gazebo>
+    <gazebo>
+        <plugin name="skid_steer_drive_controller" filename="libgazebo_ros_skid_steer_drive.so">
+            <!-- Control update rate in Hz -->
+            <updateRate>5.0</updateRate>
+            <!-- Leave empty otherwise there will be problems with sending control commands -->
+            <robotNamespace> </robotNamespace>
+            <!-- Robot kinematics -->
+            <leftFrontJoint>front_left_wheel_joint</leftFrontJoint>
+            <rightFrontJoint>front_right_wheel_joint</rightFrontJoint>
+            <leftRearJoint>rear_left_wheel_joint</leftRearJoint>
+            <rightRearJoint>rear_right_wheel_joint</rightRearJoint>
+            <wheelSeparation>0.65</wheelSeparation>
+            <wheelDiameter>0.2</wheelDiameter>
+            <!-- Maximum torque which the wheels can produce, in Nm, defaults to 5 Nm -->
+            <torque>1000</torque>
+            <!-- Topic to reveive -->
+            <commandTopic>cmd_vel</commandTopic>
+            <odometryTopic>odom</odometryTopic>
+            <odometryFrame>odom</odometryFrame>
+            <robotBaseFrame>base_link</robotBaseFrame>
+            <publishWheelTF>true</publishWheelTF>
+            <publishOdom>true</publishOdom>
+            <publishJointState>true</publishJointState>
+            <covariance_x>0.0001</covariance_x>
+            <covariance_y>0.0001</covariance_y>
+            <covariance_yaw>0.01</covariance_yaw>
+        </plugin>
+    </gazebo>
 </robot>

File: src/ford_bot/description/lidar.xacro (robot description, xacro)
@@ -25,31 +25,33 @@
         </link>
         <gazebo reference="laser_frame">
-        <material>Gazebo/Black</material>
-            <sensor name="laser" type="ray">
-                <pose> 0 0 0 0 0 0 </pose>
-                <visualize>true</visualize>
-                <update_rate>10</update_rate>
-                <ray>
-                    <scan>
-                        <horizontal>
-                            <samples>360</samples>
-                            <resolution>1</resolution>
-                            <min_angle>-3.14</min_angle>
-                            <max_angle>3.14</max_angle>
-                        </horizontal>
-                    </scan>
-                    <range>
-                        <min>0.3</min>
-                        <max>12</max>
-                        <resolution>0.04</resolution>
-                    </range>
-                </ray>
-                <plugin name="laser_controller" filename="libgazebo_ros_ray_sensor.so">
-                    <ros>
-                        <argument>~/out:=/scan</argument>
-                    </ros>
-                    <output_type>sensor_msgs/LaserScan</output_type>
-                    <frame_name>laser_frame</frame_name>
-                </plugin>
+            <material>Gazebo/FlatBlack</material>
+            <sensor type="ray" name="lidar_sensor">
+            <pose>0 0 0 0 0 0</pose>
+            <visualize>true</visualize>
+            <update_rate>5</update_rate>
+            <ray>
+                <scan>
+                    <horizontal>
+                        <samples>360</samples>
+                        <resolution>1</resolution>
+                        <min_angle>0.0</min_angle>
+                        <max_angle>6.28319</max_angle>
+                    </horizontal>
+                </scan>
+                <range>
+                    <min>0.120</min>
+                    <max>3.5</max>
+                    <resolution>0.015</resolution>
+                </range>
+                <noise>
+                    <type>gaussian</type>
+                    <mean>0.0</mean>
+                    <stddev>0.01</stddev>
+                </noise>
+            </ray>
+            <plugin name="gazebo_ros_lidar_controller" filename="libgazebo_ros_laser.so">
+                <topicName>scan</topicName>
+                <frameName>laser_frame</frameName>
+            </plugin>
             </sensor>
         </gazebo>
