Commit message: Fixed issue where the world would move in RViz instead of the robot due to the odom TF not being published properly. Issue was fixed after adding <broadcastTF> to gazebo_params.xacro file and setting it to true. Now odom is shown in the fixed frame section of RViz which allows the robot to move instead of the world around it.

File: src/ford_bot/description/gazebo_params.xacro (robot description, xacro)
@@ -30,5 +30,5 @@
         <plugin name="skid_steer_drive_controller" filename="libgazebo_ros_skid_steer_drive.so">
             <!-- Control update rate in Hz -->
-            <updateRate>5.0</updateRate>
+            <updateRate>100.0</updateRate>
             <!-- Leave empty otherwise there will be problems with sending control commands -->
             <robotNamespace> </robotNamespace>
@@ -41,13 +41,15 @@
             <wheelDiameter>0.2</wheelDiameter>
             <!-- Maximum torque which the wheels can produce, in Nm, defaults to 5 Nm -->
-            <torque>1000</torque>
-            <!-- Topic to reveive -->
+            <torque>100</torque>
+            <!-- Topic to receive -->
             <commandTopic>cmd_vel</commandTopic>
             <odometryTopic>odom</odometryTopic>
             <odometryFrame>odom</odometryFrame>
             <robotBaseFrame>base_link</robotBaseFrame>
-            <publishWheelTF>true</publishWheelTF>
+            <broadcastTF>true</broadcastTF>
+            <!-- <publishWheelTF>true</publishWheelTF>
             <publishOdom>true</publishOdom>
-            <publishJointState>true</publishJointState>
+            <publishOdomFrame>true</publishOdomFrame>
+            <publishJointState>true</publishJointState> -->
             <covariance_x>0.0001</covariance_x>
             <covariance_y>0.0001</covariance_y>

File: src/ford_bot/description/lidar.xacro (robot description, xacro)
@@ -3,9 +3,9 @@
     <joint name="laser_joint" type="fixed">
         <parent link="chassis"/>
-        <child link="laser_frame"/>
+        <child link="lidar_link"/>
         <origin xyz="0.27 0 0.07" rpy="0 0 0"/>
     </joint>
-    <link name="laser_frame">
-            <visual name="">
+    <link name="lidar_link">
+            <visual>
                 <origin xyz="0.0 0.0 0.0" rpy="0.0 0.0 0.0"/>
                 <geometry>
@@ -20,38 +20,38 @@
                 </geometry>
             </collision>
-            <xacro:inertial_cylinder mass="0.5" length="0.04" radius="0.05">
+            <xacro:inertial_cylinder mass="1" radius="0.05" length="0.04">
                 <origin xyz="0.0 0.0 0.0" rpy="0.0 0.0 0.0"/>
             </xacro:inertial_cylinder>
         </link>
-        <gazebo reference="laser_frame">
+        <gazebo reference="lidar_link">
             <material>Gazebo/FlatBlack</material>
             <sensor type="ray" name="lidar_sensor">
-            <pose>0 0 0 0 0 0</pose>
-            <visualize>true</visualize>
-            <update_rate>5</update_rate>
-            <ray>
-                <scan>
-                    <horizontal>
-                        <samples>360</samples>
-                        <resolution>1</resolution>
-                        <min_angle>0.0</min_angle>
-                        <max_angle>6.28319</max_angle>
-                    </horizontal>
-                </scan>
-                <range>
-                    <min>0.120</min>
-                    <max>3.5</max>
-                    <resolution>0.015</resolution>
-                </range>
-                <noise>
-                    <type>gaussian</type>
-                    <mean>0.0</mean>
-                    <stddev>0.01</stddev>
-                </noise>
-            </ray>
-            <plugin name="gazebo_ros_lidar_controller" filename="libgazebo_ros_laser.so">
-                <topicName>scan</topicName>
-                <frameName>laser_frame</frameName>
-            </plugin>
+                <pose>0 0 0 0 0 0</pose>
+                <visualize>true</visualize>
+                <update_rate>5</update_rate>
+                <ray>
+                    <scan>
+                        <horizontal>
+                            <samples>360</samples>
+                            <resolution>1</resolution>
+                            <min_angle>-3.14</min_angle>
+                            <max_angle>3.14</max_angle>
+                        </horizontal>
+                    </scan>
+                    <range>
+                        <min>0.3</min>
+                        <max>12</max>
+                        <resolution>0.01</resolution>
+                    </range>
+                    <!-- <noise>
+                        <type>gaussian</type>
+                        <mean>0.0</mean>
+                        <stddev>0.01</stddev>
+                    </noise> -->
+                </ray>
+                <plugin name="gazebo_ros_lidar_controller" filename="libgazebo_ros_laser.so">
+                    <topicName>scan</topicName>
+                    <frameName>lidar_link</frameName>
+                </plugin>
             </sensor>
         </gazebo>

File: src/ford_bot/description/robot_core.xacro (robot description, xacro)
@@ -3,4 +3,5 @@
     <xacro:include filename="inertial_macros.xacro"/>
     <xacro:include filename="gazebo_params.xacro"/>
+    <!-- <xacro:include filename="lidar.xacro"/> -->
     <material name="white">
         <color rgba="1 1 1 1" />
@@ -18,14 +19,14 @@
         <color rgba="1 0 0 1"/>
     </material>
+    <!-- WORLD LINK -->
+    <!-- <link name="world">
+    </link>
+ -->
     <!-- BASE LINK -->
+    <!-- <joint name="world_joint" type="fixed">
+        <parent link="world"/>
+        <child link="base_link"/>
+    </joint> -->
     <link name="base_link">
-    </link>
-    <!-- BASE_FOOTPRINT LINK -->
-    <joint name="base_footprint_joint" type="fixed">
-        <parent link="base_link"/>
-        <child link="base_footprint"/>
-        <origin xyz="0 0 0"/>
-    </joint>
-    <link name="base_footprint">
     </link>
     <!-- CHASSIS LINK -->
@@ -55,7 +56,14 @@
        <!-- All Wheel links and joints -->
     <xacro:macro name="wheel" params="name x y z">
+        <joint name="${name}_wheel_joint" type="continuous">
+            <origin xyz="${x} ${y} ${z}" rpy="-${pi/2} 0.0 0.0"/>
+            <parent link="chassis"/>
+            <child link="${name}_wheel"/>
+            <limit effort="1000.0" velocity="5.0"/>
+            <axis xyz="0.0 0.0 1"/>
+        </joint>
         <link name="${name}_wheel">
             <visual name="">
-                <origin xyz="0.0 0.0 0.0" rpy="1.57 0.0 0.0"/>
+                <origin xyz="0.0 0.0 0.0" rpy="0.0 0.0 0.0"/>
                 <geometry>
                     <cylinder radius="0.1" length="0.05"/>
@@ -66,5 +74,5 @@
             </visual>
             <collision>
-                <origin xyz="0.0 0.0 0.0" rpy="1.57 0.0 0.0"/>
+                <origin xyz="0.0 0.0 0.0" rpy="0.0 0.0 0.0"/>
                 <geometry>
                     <cylinder radius="0.1" length="0.05"/>
@@ -72,14 +80,7 @@
             </collision>
             <xacro:inertial_cylinder mass="0.75" length="0.05" radius="0.1">
-                <origin xyz="0.0 0.0 0.0" rpy="1.57 0.0 0.0"/>
+                <origin xyz="0.0 0.0 0.0" rpy="0.0 0.0 0.0"/>
             </xacro:inertial_cylinder>
         </link>
-        <joint name="${name}_wheel_joint" type="continuous">
-            <origin xyz="${x} ${y} ${z}" rpy="0 0.0 0.0"/>
-            <parent link="chassis"/>
-            <child link="${name}_wheel"/>
-            <limit effort="1000.0" velocity="5.0"/>
-            <axis xyz=".0 1.0 0.0"/>
-        </joint>
     </xacro:macro>
     <!-- Wheel Creating using macros -->
