Commit message: Added changes

File: src/ford_bot/description/lidar.xacro (robot description, xacro)
@@ -29,5 +29,5 @@
                 <pose>0 0 0 0 0 0</pose>
                 <visualize>true</visualize>
-                <update_rate>5</update_rate>
+                <update_rate>30</update_rate>
                 <ray>
                     <scan>

File: src/ford_bot/description/robot_core.xacro (robot description, xacro)
@@ -19,14 +19,14 @@
         <color rgba="1 0 0 1"/>
     </material>
-    <!-- WORLD LINK -->
-    <!-- <link name="world">
+    <!-- BASE LINK -->
+    <link name="base_link">
     </link>
- -->
-    <!-- BASE LINK -->
-    <!-- <joint name="world_joint" type="fixed">
-        <parent link="world"/>
-        <child link="base_link"/>
-    </joint> -->
-    <link name="base_link">
+    <!-- BASE FOOTRPRINT LINK-->
+    <joint name="base_footprint_joint" type="fixed">
+        <parent link="base_link"/>
+        <child link="base_footprint_link"/>
+        <origin xyz="0.0 0.0 0.0"/>
+    </joint>
+    <link name="base_footprint_link">
     </link>
     <!-- CHASSIS LINK -->
